File: hardware/OTP_generator.kicad_sch (KiCad schematic)
At the start: 4 parts, among them SW1 SW_Push, U1 ESP32-DEVKIT-V1

Commit message: Update symbols and footprints.
Parts:
- added BT1: Battery_Cell, ENAC_robotique:BatteryHolder_Keystone_1042_1x18650, symbol ENAC_robotique:Battery_Cell
- added D1, D2: D, symbol Device:D
- DS1: footprint Display:WC1602A -> ENAC_robotique:WC1602A
Connections:
- net +5V: now also U1.30 (VIN), D1.1 (K), D2.1 (K)
- net GND: now also BT1.2 (-)
- new net VBAT: BT1.1 (+)
- new net VIN: D2.2 (A)
- new net VOUT: D1.2 (A)
- no-connect marks 14 -> 15
Changed lines of the file:
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@@
 (kicad_sch (version 20230121) (generator eeschema)
   (paper "A4")
+  (junction (at 67.31 50.8) (diameter 0) (color 0 0 0 0)
+  )
   (no_connect (at 158.75 78.74))
   (no_connect (at 158.75 109.22))
@@
   (no_connect (at 128.27 91.44))
   (no_connect (at 234.95 88.9))
+  (no_connect (at 128.27 71.12))
   (no_connect (at 128.27 78.74))
   (no_connect (at 234.95 86.36))
   (no_connect (at 128.27 96.52))
   (no_connect (at 128.27 99.06))
+  (wire (pts (xy 50.8 50.8) (xy 57.15 50.8))
+    (stroke (width 0) (type default))
+  )
+  (wire (pts (xy 58.42 62.23) (xy 58.42 58.42))
+    (stroke (width 0) (type default))
+  )
   (wire (pts (xy 226.06 91.44) (xy 234.95 91.44))
     (stroke (width 0) (type default))
@@
     (stroke (width 0) (type default))
   )
+  (wire (pts (xy 67.31 50.8) (xy 74.93 50.8))
+    (stroke (width 0) (type default))
+  )
+  (wire (pts (xy 123.19 68.58) (xy 128.27 68.58))
+    (stroke (width 0) (type default))
+  )
   (wire (pts (xy 226.06 73.66) (xy 234.95 73.66))
     (stroke (width 0) (type default))
   )
+  (wire (pts (xy 64.77 50.8) (xy 67.31 50.8))
+    (stroke (width 0) (type default))
+  )
   (wire (pts (xy 245.11 60.96) (xy 245.11 63.5))
     (stroke (width 0) (type default))
   )
+  (wire (pts (xy 50.8 54.61) (xy 57.15 54.61))
+    (stroke (width 0) (type default))
+  )
   (wire (pts (xy 158.75 101.6) (xy 167.64 101.6))
     (stroke (width 0) (type default))
@@
     (stroke (width 0) (type default))
   )
+  (wire (pts (xy 58.42 58.42) (xy 50.8 58.42))
+    (stroke (width 0) (type default))
+  )
+  (wire (pts (xy 67.31 54.61) (xy 64.77 54.61))
+    (stroke (width 0) (type default))
+  )
   (wire (pts (xy 226.06 99.06) (xy 234.95 99.06))
     (stroke (width 0) (type default))
   )
   (wire (pts (xy 226.06 71.12) (xy 234.95 71.12))
+    (stroke (width 0) (type default))
+  )
+  (wire (pts (xy 67.31 50.8) (xy 67.31 54.61))
     (stroke (width 0) (type default))
   )
@@
     (effects (font (size 1.27 1.27)) (justify left bottom))
   )
+  (label "VBAT" (at 50.8 58.42 0) (fields_autoplaced)
+    (effects (font (size 1.27 1.27)) (justify left bottom))
+  )
   (label "LCD_D6" (at 167.64 106.68 180) (fields_autoplaced)
     (effects (font (size 1.27 1.27)) (justify right bottom))
@@
     (effects (font (size 1.27 1.27)) (justify right bottom))
   )
+  (label "VOUT" (at 50.8 50.8 0) (fields_autoplaced)
+    (effects (font (size 1.27 1.27)) (justify left bottom))
+  )
   (label "LCD_E" (at 226.06 68.58 0) (fields_autoplaced)
     (effects (font (size 1.27 1.27)) (justify left bottom))
@@
   (label "LCD_D7" (at 167.64 104.14 180) (fields_autoplaced)
     (effects (font (size 1.27 1.27)) (justify right bottom))
+  )
+  (label "VIN" (at 50.8 54.61 0) (fields_autoplaced)
+    (effects (font (size 1.27 1.27)) (justify left bottom))
   )
   (symbol (lib_id "ENAC_robotique:ESP32-DEVKIT-V1") (at 143.51 93.98 0) (unit 1)
@@
       (effects (font (size 1.27 1.27)) (justify left))
     )
-    (property "Footprint" "Display:WC1602A" (at 245.11 106.68 0)
+    (property "Footprint" "ENAC_robotique:WC1602A" (at 245.11 106.68 0)
       (effects (font (size 1.27 1.27) italic) hide)
     )
@@
     )
   )
+  (symbol (lib_id "Device:D") (at 60.96 50.8 180) (unit 1)
+    (in_bom yes) (on_board yes) (dnp no)
+    (property "Reference" "D1" (at 58.42 52.07 0)
+      (effects (font (size 1.27 1.27)))
+    )
+    (property "Value" "D" (at 63.5 52.07 0)
+      (effects (font (size 1.27 1.27)))
+    )
+    (property "Footprint" "" (at 60.96 50.8 0)
+      (effects (font (size 1.27 1.27)) hide)
+    )
+    (property "Datasheet" "~" (at 60.96 50.8 0)
+      (effects (font (size 1.27 1.27)) hide)
+    )
+    (property "Sim.Device" "D" (at 60.96 50.8 0)
+      (effects (font (size 1.27 1.27)) hide)
+    )
+    (property "Sim.Pins" "1=K 2=A" (at 60.96 50.8 0)
+      (effects (font (size 1.27 1.27)) hide)
+    )
+    (pin "1")
+    (pin "2")
+    (instances
+      (project "OTP_generator"
+        (path "/6b66c776-b4a0-4030-8dc1-1783907d3c0e"
+          (reference "D1") (unit 1)
+        )
+      )
+    )
+  )
+  (symbol (lib_id "power:+5V") (at 74.93 50.8 270) (unit 1)
+    (in_bom yes) (on_board yes) (dnp no) (fields_autoplaced)
+    (property "Reference" "#PWR012" (at 71.12 50.8 0)
+      (effects (font (size 1.27 1.27)) hide)
+    )
+    (property "Value" "+5V" (at 78.74 50.8 90)
+      (effects (font (size 1.27 1.27)) (justify left))
+    )
+    (property "Footprint" "" (at 74.93 50.8 0)
+      (effects (font (size 1.27 1.27)) hide)
+    )
+    (property "Datasheet" "" (at 74.93 50.8 0)
+      (effects (font (size 1.27 1.27)) hide)
+    )
+    (pin "1")
+    (instances
+      (project "OTP_generator"
+        (path "/6b66c776-b4a0-4030-8dc1-1783907d3c0e"
+          (reference "#PWR012") (unit 1)
+        )
+      )
+    )
+  )
+  (symbol (lib_id "power:+5V") (at 123.19 68.58 90) (unit 1)
+    (in_bom yes) (on_board yes) (dnp no) (fields_autoplaced)
+    (property "Reference" "#PWR013" (at 127 68.58 0)
+      (effects (font (size 1.27 1.27)) hide)
+    )
+    (property "Value" "+5V" (at 119.38 68.58 90)
+      (effects (font (size 1.27 1.27)) (justify left))
+    )
+    (property "Footprint" "" (at 123.19 68.58 0)
+      (effects (font (size 1.27 1.27)) hide)
+    )
+    (property "Datasheet" "" (at 123.19 68.58 0)
+      (effects (font (size 1.27 1.27)) hide)
+    )
+    (pin "1")
+    (instances
+      (project "OTP_generator"
+        (path "/6b66c776-b4a0-4030-8dc1-1783907d3c0e"
+          (reference "#PWR013") (unit 1)
+        )
+      )
+    )
+  )
+  (symbol (lib_id "ENAC_robotique:Battery_Cell") (at 58.42 64.77 0) (unit 1)
+    (in_bom yes) (on_board yes) (dnp no)
+    (property "Reference" "BT1" (at 60.96 62.23 0)
+      (effects (font (size 1.27 1.27)) (justify left))
+    )
+    (property "Value" "Battery_Cell" (at 60.96 66.04 0)
+      (effects (font (size 1.27 1.27)) (justify left))
+    )
+    (property "Footprint" "ENAC_robotique:BatteryHolder_Keystone_1042_1x18650" (at 58.42 64.516 90)
+      (effects (font (size 1.27 1.27)) hide)
+    )
+    (property "Datasheet" "~" (at 58.42 64.516 90)
+      (effects (font (size 1.27 1.27)) hide)
+    )
+    (pin "1")
+    (pin "2")
+    (instances
+      (project "OTP_generator"
+        (path "/6b66c776-b4a0-4030-8dc1-1783907d3c0e"
+          (reference "BT1") (unit 1)
+        )
+      )
+    )
+  )
   (symbol (lib_id "power:GND") (at 158.75 116.84 90) (unit 1)
     (in_bom yes) (on_board yes) (dnp no) (fields_autoplaced)
@@
     )
   )
+  (symbol (lib_id "Device:D") (at 60.96 54.61 180) (unit 1)
+    (in_bom yes) (on_board yes) (dnp no)
+    (property "Reference" "D2" (at 58.42 55.88 0)
+      (effects (font (size 1.27 1.27)))
+    )
+    (property "Value" "D" (at 63.5 55.88 0)
+      (effects (font (size 1.27 1.27)))
+    )
+    (property "Footprint" "" (at 60.96 54.61 0)
+      (effects (font (size 1.27 1.27)) hide)
+    )
+    (property "Datasheet" "~" (at 60.96 54.61 0)
+      (effects (font (size 1.27 1.27)) hide)
+    )
+    (property "Sim.Device" "D" (at 60.96 54.61 0)
+      (effects (font (size 1.27 1.27)) hide)
+    )
+    (property "Sim.Pins" "1=K 2=A" (at 60.96 54.61 0)
+      (effects (font (size 1.27 1.27)) hide)
+    )
+    (pin "1")
+    (pin "2")
+    (instances
+      (project "OTP_generator"
+        (path "/6b66c776-b4a0-4030-8dc1-1783907d3c0e"
+          (reference "D2") (unit 1)
+        )
+      )
+    )
+  )
   (symbol (lib_id "power:GND") (at 158.75 119.38 90) (unit 1)
     (in_bom yes) (on_board yes) (dnp no) (fields_autoplaced)
@@
         )
       )
+    )
+  )
+  (symbol (lib_id "power:GND") (at 58.42 67.31 0) (unit 1)
+    (in_bom yes) (on_board yes) (dnp no) (fields_autoplaced)
+    (property "Reference" "#PWR011" (at 58.42 73.66 0)
+      (effects (font (size 1.27 1.27)) hide)
+    )
+    (property "Value" "GND" (at 58.42 72.39 0)
+      (effects (font (size 1.27 1.27)))
+    )
+    (property "Footprint" "" (at 58.42 67.31 0)
+      (effects (font (size 1.27 1.27)) hide)
+    )
+    (property "Datasheet" "" (at 58.42 67.31 0)
+      (effects (font (size 1.27 1.27)) hide)
+    )
+    (pin "1")
+    (instances
+      (project "OTP_generator"
+        (path "/6b66c776-b4a0-4030-8dc1-1783907d3c0e"
+          (reference "#PWR011") (unit 1)
+        )
+      )
